Commit message: うーん

File: src/meistar_description/urdf/robot.urdf.xacro (robot description, xacro)
@@ -1,4 +1,11 @@
 <?xml version="1.0"?>
 <robot name="meistar_bot" xmlns:xacro="http://www.ros.org/wiki/xacro">
+  <!-- Materials -->
+  <material name="blue">
+    <color rgba="0 0 0.8 1"/>
+  </material>
+  <material name="grey">
+    <color rgba="0.5 0.5 0.5 1"/>
+  </material>
   <!-- Base Link -->
   <link name="base_link">
@@ -7,7 +14,5 @@
         <box size="0.5 0.5 0.2"/>
       </geometry>
-      <material name="blue">
-        <color rgba="0 0 1 1"/>
-      </material>
+      <material name="blue"/>
     </visual>
     <collision>
@@ -18,5 +23,5 @@
     <inertial>
       <mass value="10.0"/>
-      <origin xyz="0 0 0"/>
+      <origin xyz="0 0 0" rpy="0 0 0"/>
       <inertia ixx="0.2" ixy="0" ixz="0" iyy="0.2" iyz="0" izz="0.4"/>
     </inertial>
@@ -28,8 +33,11 @@
         <cylinder radius="0.05" length="0.1"/>
       </geometry>
-      <material name="black">
-        <color rgba="0 0 0 1"/>
-      </material>
+      <material name="grey"/>
     </visual>
+    <collision>
+      <geometry>
+        <cylinder radius="0.05" length="0.1"/>
+      </geometry>
+    </collision>
   </link>
   <joint name="lidar_joint" type="fixed">
@@ -45,14 +53,17 @@
   <gazebo>
     <plugin
-      filename="gz-sim-planar-move-system"
-      name="gz::sim::systems::PlanarMove">
+      filename="gz-sim-velocity-control-system"
+      name="gz::sim::systems::VelocityControl">
       <topic>/model/meistar_bot/cmd_vel</topic>
-      <odom_publish_frequency>50</odom_publish_frequency>
+    </plugin>
+  </gazebo>
+  <gazebo>
+    <plugin filename="gz-sim-odometry-publisher-system"
+            name="gz::sim::systems::OdometryPublisher">
+      <odom_frame>odom</odom_frame>
+      <robot_base_frame>base_link</robot_base_frame>
       <odom_topic>/model/meistar_bot/odometry</odom_topic>
       <tf_topic>/model/meistar_bot/tf</tf_topic>
-      <frame_id>odom</frame_id>
-      <child_frame_id>base_link</child_frame_id>
-      <publish_odom>true</publish_odom>
-      <publish_odom_tf>true</publish_odom_tf>
+      <dimensions>3</dimensions>
     </plugin>
   </gazebo>
@@ -60,5 +71,4 @@
   <gazebo reference="lidar_link">
     <sensor name="lidar" type="gpu_lidar">
-      <gz_frame_id>lidar_link</gz_frame_id>
       <topic>scan</topic>
       <update_rate>10</update_rate>
@@ -73,8 +83,10 @@
         </scan>
         <range>
-          <min>0.1</min>
-          <max>12.0</max>
+          <min>0.08</min>
+          <max>10.0</max>
+          <resolution>0.01</resolution>
         </range>
       </lidar>
+      <always_on>1</always_on>
       <visualize>true</visualize>
     </sensor>

Commit message: リファクタリング

File: src/meistar_description/urdf/robot.urdf.xacro (robot description, xacro)
@@ -1,96 +1,7 @@
 <?xml version="1.0"?>
 <robot name="meistar_bot" xmlns:xacro="http://www.ros.org/wiki/xacro">
-  <!-- Materials -->
-  <material name="blue">
-    <color rgba="0 0 0.8 1"/>
-  </material>
-  <material name="grey">
-    <color rgba="0.5 0.5 0.5 1"/>
-  </material>
-  <!-- Base Link -->
-  <link name="base_link">
-    <visual>
-      <geometry>
-        <box size="0.5 0.5 0.2"/>
-      </geometry>
-      <material name="blue"/>
-    </visual>
-    <collision>
-      <geometry>
-        <box size="0.5 0.5 0.2"/>
-      </geometry>
-    </collision>
-    <inertial>
-      <mass value="10.0"/>
-      <origin xyz="0 0 0" rpy="0 0 0"/>
-      <inertia ixx="0.2" ixy="0" ixz="0" iyy="0.2" iyz="0" izz="0.4"/>
-    </inertial>
-  </link>
-  <!-- Lidar Link -->
-  <link name="lidar_link">
-    <visual>
-      <geometry>
-        <cylinder radius="0.05" length="0.1"/>
-      </geometry>
-      <material name="grey"/>
-    </visual>
-    <collision>
-      <geometry>
-        <cylinder radius="0.05" length="0.1"/>
-      </geometry>
-    </collision>
-  </link>
-  <joint name="lidar_joint" type="fixed">
-    <parent link="base_link"/>
-    <child link="lidar_link"/>
-    <origin xyz="0 0 0.15" rpy="0 0 0"/>
-  </joint>
-  <gazebo reference="base_link">
-    <mu1>0.0</mu1>
-    <mu2>0.0</mu2>
-  </gazebo>
-  <!-- Gazebo Plugins (Gazebo Harmonic / GZ Sim) -->
-  <gazebo>
-    <!-- Movement control -->
-    <plugin
-      filename="gz-sim-velocity-control-system"
-      name="gz::sim::systems::VelocityControl">
-      <topic>/model/meistar_bot/cmd_vel</topic>
-    </plugin>
-    <!-- Odometry and TF publishing -->
-    <plugin
-      filename="gz-sim-odometry-publisher-system"
-      name="gz::sim::systems::OdometryPublisher">
-      <odom_topic>/model/meistar_bot/odometry</odom_topic>
-      <tf_topic>/model/meistar_bot/tf</tf_topic>
-      <odom_publish_frequency>50</odom_publish_frequency>
-      <odom_frame>odom</odom_frame>
-      <robot_base_frame>base_link</robot_base_frame>
-    </plugin>
-  </gazebo>
-  <!-- Lidar Sensor -->
-  <gazebo reference="lidar_link">
-    <sensor name="lidar" type="gpu_lidar">
-      <topic>/scan</topic>
-      <update_rate>10</update_rate>
-      <gz_frame_id>lidar_link</gz_frame_id>
-      <lidar>
-        <scan>
-          <horizontal>
-            <samples>640</samples>
-            <resolution>1</resolution>
-            <min_angle>-3.14</min_angle>
-            <max_angle>3.14</max_angle>
-          </horizontal>
-        </scan>
-        <range>
-          <min>0.08</min>
-          <max>10.0</max>
-          <resolution>0.01</resolution>
-        </range>
-      </lidar>
-      <always_on>1</always_on>
-      <visualize>false</visualize>
-    </sensor>
-  </gazebo>
+  <!-- Include component Xacro files -->
+  <xacro:include filename="chassis.xacro" />
+  <xacro:include filename="lidar.xacro" />
+  <xacro:include filename="gazebo.xacro" />
 </robot>
