Commit message: Refactor robot to 6-wheel rover and update kinematics
- Modified `chassis.xacro` to resize the base and added 6 wheels using a macro.
- Replaced `VelocityControl` with `DiffDrive` in `gazebo.xacro` to enable skid-steer control for the 6 wheels.
- Updated Nav2 config (`mapping_nav_params.yaml`) to use `DifferentialMotionModel` and disabled Y-axis velocity (strafe) to match the new non-holonomic kinematics.

Co-authored-by: sosukigara <219259772+sosukigara@users.noreply.github.com>

File: src/meistar_description/urdf/chassis.xacro (robot description, xacro)
@@ -8,4 +8,7 @@
     <color rgba="0.0 0.8 1.0 1"/>
   </material>
+  <material name="black">
+    <color rgba="0.1 0.1 0.1 1"/>
+  </material>
   <!-- Base Link -->
   <link name="base_link">
@@ -13,5 +16,6 @@
       <origin xyz="0 0 0" rpy="0 0 0"/>
       <geometry>
-        <box size="0.5 0.5 0.2"/>
+        <!-- Modified to look more like a rover chassis -->
+        <box size="0.6 0.4 0.15"/>
       </geometry>
       <material name="carbon_grey"/>
@@ -19,7 +23,7 @@
     <!-- Accent Visual (Decorative strip) -->
     <visual>
-      <origin xyz="0.251 0 0.05" rpy="0 0 0"/>
+      <origin xyz="0.301 0 0.03" rpy="0 0 0"/>
       <geometry>
-        <box size="0.01 0.4 0.02"/>
+        <box size="0.01 0.3 0.02"/>
       </geometry>
       <material name="neon_blue"/>
@@ -27,5 +31,5 @@
     <collision>
       <geometry>
-        <box size="0.5 0.5 0.2"/>
+        <box size="0.6 0.4 0.15"/>
       </geometry>
     </collision>
@@ -44,7 +48,54 @@
       </material>
     </visual>
-    <mu1>0.0</mu1>
-    <mu2>0.0</mu2>
   </gazebo>
+  <!-- Wheel Macro -->
+  <xacro:macro name="wheel" params="prefix suffix x y">
+    <link name="${prefix}_${suffix}_wheel">
+      <visual>
+        <!-- rotate cylinder to lay flat along Y axis -->
+        <origin xyz="0 0 0" rpy="${pi/2} 0 0"/>
+        <geometry>
+          <cylinder radius="0.1" length="0.05"/>
+        </geometry>
+        <material name="black"/>
+      </visual>
+      <collision>
+        <origin xyz="0 0 0" rpy="${pi/2} 0 0"/>
+        <geometry>
+          <cylinder radius="0.1" length="0.05"/>
+        </geometry>
+      </collision>
+      <inertial>
+        <mass value="1.0"/>
+        <origin xyz="0 0 0" rpy="${pi/2} 0 0"/>
+        <!-- Rough inertia for cylinder -->
+        <inertia ixx="0.01" ixy="0" ixz="0" iyy="0.01" iyz="0" izz="0.01"/>
+      </inertial>
+    </link>
+    <joint name="${prefix}_${suffix}_joint" type="continuous">
+      <parent link="base_link"/>
+      <child link="${prefix}_${suffix}_wheel"/>
+      <!-- Wheel offset from center. Z = -0.05 drops the wheels down a bit -->
+      <origin xyz="${x} ${y} -0.05" rpy="0 0 0"/>
+      <axis xyz="0 1 0"/>
+    </joint>
+    <gazebo reference="${prefix}_${suffix}_wheel">
+      <mu1>1.0</mu1>
+      <mu2>0.1</mu2>
+      <material>
+        <ambient>0.0 0.0 0.0 1</ambient>
+        <diffuse>0.0 0.0 0.0 1</diffuse>
+        <specular>0.1 0.1 0.1 1</specular>
+      </material>
+    </gazebo>
+  </xacro:macro>
+  <!-- 6 Wheels: Left side -->
+  <xacro:wheel prefix="front" suffix="left" x="0.25" y="0.25" />
+  <xacro:wheel prefix="middle" suffix="left" x="0.0" y="0.25" />
+  <xacro:wheel prefix="rear" suffix="left" x="-0.25" y="0.25" />
+  <!-- 6 Wheels: Right side -->
+  <xacro:wheel prefix="front" suffix="right" x="0.25" y="-0.25" />
+  <xacro:wheel prefix="middle" suffix="right" x="0.0" y="-0.25" />
+  <xacro:wheel prefix="rear" suffix="right" x="-0.25" y="-0.25" />
   <!-- Footprint (Ground projection) -->
   <link name="base_footprint"/>

File: src/meistar_description/urdf/gazebo.xacro (robot description, xacro)
@@ -3,8 +3,17 @@
   <!-- Gazebo Plugins (Gazebo Harmonic / GZ Sim) -->
   <gazebo>
-    <!-- Movement control -->
+    <!-- Skid Steer Diff Drive Control for 6 wheels -->
     <plugin
-      filename="gz-sim-velocity-control-system"
-      name="gz::sim::systems::VelocityControl">
+      filename="gz-sim-diff-drive-system"
+      name="gz::sim::systems::DiffDrive">
+      <left_joint>front_left_joint</left_joint>
+      <left_joint>middle_left_joint</left_joint>
+      <left_joint>rear_left_joint</left_joint>
+      <right_joint>front_right_joint</right_joint>
+      <right_joint>middle_right_joint</right_joint>
+      <right_joint>rear_right_joint</right_joint>
+      <wheel_separation>0.5</wheel_separation>
+      <wheel_radius>0.1</wheel_radius>
+      <odom_publish_frequency>50</odom_publish_frequency>
       <topic>/model/meistar_bot/cmd_vel</topic>
     </plugin>

Commit message: Upgrade to 6-wheel steer and advanced Nav2 plugins
- Updated URDF `chassis.xacro` to add a Z-axis steering joint to all 6 wheels.
- Reverted to `VelocityControl` in Gazebo to allow holonomic crab-steering simulation.
- Replaced `DWBLocalPlanner` with `RegulatedPurePursuitController` to eliminate path "bulging" and enforce strict tracking.
- Replaced `NavfnPlanner` with `SmacPlanner2D` for cost-aware global planning.
- Heavily modified costmap inflation (`cost_scaling_factor: 2.0`, `inflation_radius: 3.5`) to force the robot to stay as far from walls as possible.

Co-authored-by: sosukigara <219259772+sosukigara@users.noreply.github.com>

File: src/meistar_description/urdf/chassis.xacro (robot description, xacro)
@@ -49,6 +49,23 @@
     </visual>
   </gazebo>
-  <!-- Wheel Macro -->
+  <!-- Steerable Wheel Macro -->
   <xacro:macro name="wheel" params="prefix suffix x y">
+    <!-- Steering Link (acts as the pivot/knuckle) -->
+    <link name="${prefix}_${suffix}_steer_link">
+      <inertial>
+        <mass value="0.1"/>
+        <origin xyz="0 0 0" rpy="0 0 0"/>
+        <inertia ixx="0.001" ixy="0" ixz="0" iyy="0.001" iyz="0" izz="0.001"/>
+      </inertial>
+    </link>
+    <!-- Steering Joint (rotates around Z-axis) -->
+    <joint name="${prefix}_${suffix}_steer_joint" type="revolute">
+      <parent link="base_link"/>
+      <child link="${prefix}_${suffix}_steer_link"/>
+      <origin xyz="${x} ${y} -0.05" rpy="0 0 0"/>
+      <axis xyz="0 0 1"/>
+      <limit lower="-1.57" upper="1.57" effort="10.0" velocity="2.0"/>
+    </joint>
+    <!-- Wheel Link -->
     <link name="${prefix}_${suffix}_wheel">
       <visual>
@@ -73,14 +90,15 @@
       </inertial>
     </link>
+    <!-- Drive Joint (rotates around Y-axis) -->
     <joint name="${prefix}_${suffix}_joint" type="continuous">
-      <parent link="base_link"/>
+      <parent link="${prefix}_${suffix}_steer_link"/>
       <child link="${prefix}_${suffix}_wheel"/>
-      <!-- Wheel offset from center. Z = -0.05 drops the wheels down a bit -->
-      <origin xyz="${x} ${y} -0.05" rpy="0 0 0"/>
+      <!-- Wheel is exactly at the steering pivot -->
+      <origin xyz="0 0 0" rpy="0 0 0"/>
       <axis xyz="0 1 0"/>
     </joint>
     <gazebo reference="${prefix}_${suffix}_wheel">
       <mu1>1.0</mu1>
-      <mu2>0.1</mu2>
+      <mu2>1.0</mu2> <!-- Back to 1.0 since it can steer -->
       <material>
         <ambient>0.0 0.0 0.0 1</ambient>

File: src/meistar_description/urdf/gazebo.xacro (robot description, xacro)
@@ -3,17 +3,8 @@
   <!-- Gazebo Plugins (Gazebo Harmonic / GZ Sim) -->
   <gazebo>
-    <!-- Skid Steer Diff Drive Control for 6 wheels -->
+    <!-- Holonomic Velocity Control for 6-wheel steer/drive -->
     <plugin
-      filename="gz-sim-diff-drive-system"
-      name="gz::sim::systems::DiffDrive">
-      <left_joint>front_left_joint</left_joint>
-      <left_joint>middle_left_joint</left_joint>
-      <left_joint>rear_left_joint</left_joint>
-      <right_joint>front_right_joint</right_joint>
-      <right_joint>middle_right_joint</right_joint>
-      <right_joint>rear_right_joint</right_joint>
-      <wheel_separation>0.5</wheel_separation>
-      <wheel_radius>0.1</wheel_radius>
-      <odom_publish_frequency>50</odom_publish_frequency>
+      filename="gz-sim-velocity-control-system"
+      name="gz::sim::systems::VelocityControl">
       <topic>/model/meistar_bot/cmd_vel</topic>
     </plugin>

Commit message: Fix 6-wheel steering animation in Gazebo and RViz
- Changed steer joint from `revolute` (with limits) to `continuous` to prevent wheels from getting stuck when pivoting 180 degrees.
- Added a 3cm caster offset (`xyz="-0.03 0 0"`) to the drive joint to resolve violent physics fluttering caused by zero caster trail.
- Added the `gz-sim-joint-state-publisher-system` plugin to `gazebo.xacro` so that joint rotations are published to ROS 2, restoring wheel animations in RViz.

Co-authored-by: sosukigara <219259772+sosukigara@users.noreply.github.com>

File: src/meistar_description/urdf/chassis.xacro (robot description, xacro)
@@ -60,10 +60,9 @@
     </link>
     <!-- Steering Joint (rotates around Z-axis) -->
-    <joint name="${prefix}_${suffix}_steer_joint" type="revolute">
+    <joint name="${prefix}_${suffix}_steer_joint" type="continuous">
       <parent link="base_link"/>
       <child link="${prefix}_${suffix}_steer_link"/>
       <origin xyz="${x} ${y} -0.05" rpy="0 0 0"/>
       <axis xyz="0 0 1"/>
-      <limit lower="-1.57" upper="1.57" effort="10.0" velocity="2.0"/>
     </joint>
     <!-- Wheel Link -->
@@ -94,6 +93,6 @@
       <parent link="${prefix}_${suffix}_steer_link"/>
       <child link="${prefix}_${suffix}_wheel"/>
-      <!-- Wheel is exactly at the steering pivot -->
-      <origin xyz="0 0 0" rpy="0 0 0"/>
+      <!-- Caster offset to allow stable passive steering -->
+      <origin xyz="-0.03 0 0" rpy="0 0 0"/>
       <axis xyz="0 1 0"/>
     </joint>

File: src/meistar_description/urdf/gazebo.xacro (robot description, xacro)
@@ -8,4 +8,10 @@
       name="gz::sim::systems::VelocityControl">
       <topic>/model/meistar_bot/cmd_vel</topic>
+    </plugin>
+    <!-- Joint State Publisher for RViz animation -->
+    <plugin
+      filename="gz-sim-joint-state-publisher-system"
+      name="gz::sim::systems::JointStatePublisher">
+      <topic>joint_states</topic>
     </plugin>
     <!-- Odometry and TF publishing -->

Commit message: Fix Gazebo URDF link lumping by adding dummy inertials
- Added dummy `<inertial>` tags to `base_footprint` and `lidar_link` in their respective xacro files.
- Prevents Gazebo from aggressively lumping or dropping these fixed links, which was causing the model to fail spawning (Error Code 17) and OdometryPublisher to timeout waiting for `base_footprint` TF.

Co-authored-by: sosukigara <219259772+sosukigara@users.noreply.github.com>

File: src/meistar_description/urdf/chassis.xacro (robot description, xacro)
@@ -116,5 +116,11 @@
   <xacro:wheel prefix="rear" suffix="right" x="-0.25" y="-0.25" />
   <!-- Footprint (Ground projection) -->
-  <link name="base_footprint"/>
+  <link name="base_footprint">
+    <inertial>
+      <mass value="0.001"/>
+      <origin xyz="0 0 0" rpy="0 0 0"/>
+      <inertia ixx="0.0001" ixy="0.0" ixz="0.0" iyy="0.0001" iyz="0.0" izz="0.0001"/>
+    </inertial>
+  </link>
   <joint name="base_footprint_joint" type="fixed">
     <parent link="base_footprint"/>

File: src/meistar_description/urdf/lidar.xacro (robot description, xacro)
@@ -16,4 +16,9 @@
       </geometry>
     </collision>
+    <inertial>
+      <mass value="0.1"/>
+      <origin xyz="0 0 0" rpy="0 0 0"/>
+      <inertia ixx="0.0001" ixy="0" ixz="0" iyy="0.0001" iyz="0" izz="0.0001"/>
+    </inertial>
   </link>
   <gazebo reference="lidar_link">
