Commit message: fix(nav): SLAM lifecycle のレースと lidar 自己観測を直す
slam_toolbox の activate を固定秒数の TimerAction で configure と
独立に走らせており、configure 前に activate が発火すると SLAM が
inactive のまま固まって map フレームが出ず、Nav2 の global_costmap が
configure 失敗していた。結果として pose goal が "Start occupied" または
action reject で止まっていた。OnStateTransition で inactive 到達を
待ってから activate する。

あわせて lidar を base_link の天面すぐ上 (0.15) から 0.30 へ。水平レイが
自機の箱の角を 0.17m で捉えて擬似障害物を作り、global_costmap の
inflation (radius 1.2m) がロボット自身の開始セルを埋めていた。
計測: 最小レンジ 0.170m -> 2.252m、0.6m 未満の有効点数 36 -> 0、
開始セルのコスト 253 -> 0。

File: src/meistar_description/urdf/lidar.xacro (robot description, xacro)
@@ -26,8 +26,12 @@
     </visual>
   </gazebo>
+  <!-- lidar は base_link の天面 (half-height 0.1) から十分上に離す。
+       すぐ上 (0.15) に置くと水平レイが箱の角を捉えて 0.17m の擬似障害物になり、
+       global_costmap の inflation がロボット自身の開始セルを埋めて
+       "Start occupied" になる。 -->
   <joint name="lidar_joint" type="fixed">
     <parent link="base_link"/>
     <child link="lidar_link"/>
-    <origin xyz="0 0 0.15" rpy="0 0 0"/>
+    <origin xyz="0 0 0.30" rpy="0 0 0"/>
   </joint>
   <!-- Gazebo Sensor Plugin -->

File: src/meistar_description/urdf/robot.urdf.xacro (robot description, xacro)
@@ -4,4 +4,5 @@
   <xacro:include filename="chassis.xacro" />
   <xacro:include filename="lidar.xacro" />
+  <xacro:include filename="camera.xacro" />
   <xacro:include filename="gazebo.xacro" />
 </robot>
